File: Paul-PCB-KICAD.kicad_pcb (KiCad board)
At the start: 2 copper layers, 330.9 x 105.7 mm, 173 parts, among them SW1 SW_Push, U1 ATmega32U4-AU, Y1 16MHz

Commit message: Merge of Final PCB V1 and Firmware
Firmware was on laptop and PCB on Desktop
Parts:
- added REF**: JLC_Tooling_Hole, random-keyboard-parts:JLC_Tooling_Hole, F.Cu at (296.2, -85.6)
- added REF**: JLC_Tooling_Hole, random-keyboard-parts:JLC_Tooling_Hole, F.Cu at (0.65, -87.3)
- added REF**: JLC_Tooling_Hole, random-keyboard-parts:JLC_Tooling_Hole, F.Cu at (-0.20, 2.39)
- added REF**: JLC_Tooling_Hole, random-keyboard-parts:JLC_Tooling_Hole, F.Cu at (309.0, 6.27)
- renumbered D1 to D001, D2 to D002, D3 to D003, D4 to D004, D5 to D005, D6 to D006, D7 to D007, D8 to D008, D9 to D009, D10 to D010, D11 to D011, D12 to D012, D13 to D013, D14 to D014, MX0 to MX000, MX1 to MX001, MX2 to MX002, MX3 to MX003, MX4 to MX004, MX5 to MX005, MX6 to MX006, MX7 to MX007, MX8 to MX008, MX9 to MX009, MX10 to MX010, MX11 to MX011, MX12 to MX012, MX13 to MX013, MX14 to MX014
